File: väggtermometer.kicad_pcb (KiCad board)
At the start: 2 copper layers, 35 x 191 mm, 155 parts, among them J1 USB_C_Receptacle_USB2.0, J2 Conn_01x08, J4 NC, J8 Conn_01x02, Q1 BSS84, SW1 SW_MEC_5G, SW3 SW_MEC_5G, U1 ESP32-C3, U2 RT9080, U3 TC1047AxNB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

Commit message: pictures etc
Other:
- board text removed: "Dischidia astephana"
- board text removed: "Illustration: Richard E. Rintz CC-BY"
- board text removed: "Made in Mönsterås"
