File: väggtermometer.kicad_pcb (KiCad board)
At the start: 2 copper layers, 35 x 191 mm, 155 parts, among them J1 USB_C_Receptacle_USB2.0, J2 Conn_01x08, J4 NC, J8 Conn_01x02, Q1 BSS84, SW1 SW_MEC_5G, SW3 SW_MEC_5G, U1 ESP32-C3, U2 RT9080, U3 TC1047AxNB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

Commit message: mix
Parts:
- renumbered REF** to FID1, REF** to FID2, REF** to FID3
Routing:
- net GND: vias 18 -> 17
Changed lines of the file:
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@@
 		(pad_to_mask_clearance 0)
 		(allow_soldermask_bridges_in_footprints no)
+		(aux_axis_origin 39.40901 224.59099)
 		(pcbplotparams
 			(layerselection 0x00010fc_ffffffff)
@@
 		(descr "Circular Fiducial, 1mm bare copper, 2mm soldermask opening (Level A)")
 		(tags "fiducial")
-		(property "Reference" "REF**"
+		(property "Reference" "FID1"
 			(at 0 -2 0)
 			(layer "F.SilkS")
@@
 		(descr "Circular Fiducial, 1mm bare copper, 2mm soldermask opening (Level A)")
 		(tags "fiducial")
-		(property "Reference" "REF**"
+		(property "Reference" "FID2"
 			(at 0 -2 0)
 			(layer "F.SilkS")
@@
 		(descr "Circular Fiducial, 1mm bare copper, 2mm soldermask opening (Level A)")
 		(tags "fiducial")
-		(property "Reference" "REF**"
+		(property "Reference" "FID3"
 			(at 0 -2 0)
 			(layer "F.SilkS")
@@
 	)
 	(via
-		(at 62.25 202)
-		(size 0.6)
-		(drill 0.3)
-		(layers "F.Cu" "B.Cu")
-		(net 2)
-	)
-	(via
 		(at 66 183.6)
 		(size 0.6)
@@
 			)
 		)
+	)
+	(zone
+		(net 0)
+		(net_name "")
+		(layer "F.Cu")
+		(hatch edge 0.5)
+		(connect_pads
+			(clearance 0)
+		)
+		(min_thickness 0.25)
+		(filled_areas_thickness no)
+		(keepout
+			(tracks allowed)
+			(vias allowed)
+			(pads allowed)
+			(copperpour not_allowed)
+			(footprints allowed)
+		)
+		(fill
+			(thermal_gap 0.5)
+			(thermal_bridge_width 0.5)
+		)
+		(polygon
+			(pts
+				(xy 61.3 201) (xy 63.2 201) (xy 63.2 203) (xy 61.3 203)
+			)
+		)

Commit message: info and stuff
Parts:
- moved C16 46.0 mm to (115.4, 214.8)
- moved J1 46.0 mm to (114.8, 222.7)
- moved R5 46.0 mm to (113.5, 224.2)
- moved R6 46.0 mm to (114.5, 224.2)
- moved U4 46.0 mm to (111.2, 156.2)
- moved C15 46.0 mm to (108.3, 156.4)
- moved C5 46.0 mm to (105.5, 196.0)
- moved ? 46.0 mm to (117.5, 216.2)
- moved ? 46.0 mm to (112.8, 212.9)
- moved BT1 46.0 mm to (94.8, 154.8)
- moved C1 46.0 mm to (107.3, 201.0)
- moved C10 46.0 mm to (115.6, 198.5)
- moved C11 46.0 mm to (106.0, 218.6)
- moved C12 46.0 mm to (107.8, 214.8)
- moved C13 46.0 mm to (110.8, 203.8)
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
Commit message: updates
Other:
- board text added: "CERN-OHL-P 2,0"
- board text added: "SE000028"
