File: väggtermometer.kicad_sch (KiCad schematic)
At the start: 145 parts, among them J1 USB_C_Receptacle_USB2.0, J2 Conn_01x08, J4 NC, J8 Conn_01x02, Q1 BSS84, SW1 SW_MEC_5G, SW3 SW_MEC_5G, U1 ESP32-C3, U2 RT9080, U3 TC1047AxNB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

Commit message: mix
Parts:
- R13: value 5,1kΩ -> 10kΩ
Changed lines of the file:
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@@
 			)
 		)
-		(property "Value" "5,1kΩ"
+		(property "Value" "10kΩ"
 			(at 30.48 93.98 0)
 			(effects
