File: V2_0603/termometer2.kicad_pcb (KiCad board)
At the start: 2 copper layers, 35 x 191 mm, 170 parts, among them J1 USB_C_Receptacle_USB2.0, J2 Conn_01x03, J3 Conn_01x03, Q1 BSS84, SW3 SW_MEC_5G, U1 ESP32-C3, U2 RT9080, U3 SL197-1, U4 MCP73831, U5 W25Q32RVXHJQ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

Commit message: cleanup
Parts:
- removed REF**: KiCad-Logo_5mm_SilkScreen, Symbol:KiCad-Logo_5mm_SilkScreen
- removed REF**: CE-Logo_8.5x6mm_SilkScreen, Symbol:CE-Logo_8.5x6mm_SilkScreen
- moved C21 0.30 mm to (111.5, 54.3)
- renumbered REF** to REF1, REF** to REF2
Routing:
- net +5V: track 51.7 -> 50.8 mm
- net GND: vias 25 -> 26
Other:
- board text removed: "Dischidia astephana"
- board text removed: "Illustration: Richard Rintz CC-BY"
- board text removed: "Made in Sweden"
- board text removed: "Ping"
- board text removed: "SE000028"
- board text removed: "V1,1"
- board text removed: "hobbyelektronik"
